File: Schematics-PCB-Design/aadhuNIK-Main/aadhuNIK-Main.kicad_pcb (KiCad board)
At the start: 2 copper layers, 70 parts, among them J1 Conn_01x05_Pin, J10 Conn_01x01_Pin, J2 Conn_01x06_Pin, J3 Barrel_Jack, J4 Conn_01x06_Pin, J5 Conn_01x05_Pin, J6 Barrel_Jack, J7 Conn_01x01_Pin, J8 Conn_01x01_Pin, J9 Conn_01x01_Pin, U1 LM2596S-ADJ, U10 TMC2209-LA, U11 TMC2209-LA, U12 ICM-20948, U13 LM2596S-5, U14 LM2596S-ADJ, U2 LM2596S-5, U3 TMC2209-LA, U4 TMC2209-LA, U5 ICM-20948, U6 MAX98357A, U7 MAX98357A, U8 MAX98357A, U9 MAX98357A

Commit message: Update KiCad schematic and PCB
Parts:
- removed A1: RaspberryPi_Pico, Module:RaspberryPi_Pico_Common_Unspecified
- removed C10, C16, C21: 47uF, PCM_SparkFun-Capacitor:C_0805_2012Metric
- removed C11, C12, C14, C17, C19, C22: 100uF, PCM_SparkFun-Capacitor:Panasonic_D
- removed C13: 10uF, PCM_SparkFun-Capacitor:C_0603_1608Metric_Polar
- removed C15, C20, C9: 1uF_0603_25V, PCM_4ms_Capacitor:C_0603
- removed C18: 2.2uF, PCM_SparkFun-Capacitor:C_0805_2012Metric
- removed D2, D3, D4, D5, D6: 1N5822, PCM_Diode_THT_AKL:D_DO-201AD_P12.70mm_Horizontal
- removed F1: Fuse_Polarized, Fuse:Fuse_0402_1005Metric
- removed J10, J7, J8: Conn_01x01_Pin, Connector_PinHeader_1.00mm:PinHeader_1x01_P1.00mm_Vertical
- removed J3, J6: Barrel_Jack, Connector_BarrelJack:BarrelJack_SwitchcraftConxall_RAPC10U_Horizontal
- removed J4: Conn_01x06_Pin, Connector_Harwin:Harwin_M20-89006xx_1x06_P2.54mm_Horizontal
- removed J5: Conn_01x05_Pin, Connector_Harwin:Harwin_M20-89005xx_1x05_P2.54mm_Horizontal
- removed L1, L2, L3: 1.0uH, PCM_SparkFun-Coil:0805
- removed R3, R6: 10k_0402, Resistor_SMD:R_0402_1005Metric
- removed R4, R5: 4.7k, PCM_SparkFun-Resistor:R_0402_1005Metric
- removed U10, U11, U3, U4: TMC2209-LA, Package_DFN_QFN:VQFN-28-1EP_5x5mm_P0.5mm_EP3.7x3.7mm_ThermalVias
- removed U12, U5: ICM-20948, Sensor_Motion:InvenSense_QFN-24_3x3mm_P0.4mm
- removed U13: LM2596S-5, PCM_Package_TO_SOT_SMD_AKL:TO-263-4_ThermalVias
- removed U14: LM2596S-ADJ, Package_TO_SOT_SMD:TO-263-5_TabPin3
- removed U6, U7, U8, U9: MAX98357A, Package_DFN_QFN:TQFN-16-1EP_3x3mm_P0.5mm_EP1.23x1.23mm
- added C28: 100uF, PCM_SparkFun-Capacitor:Panasonic_D, F.Cu at (129.0, 91.4)
- added C30: 1.0uF, PCM_SparkFun-Capacitor:C_0402_1005Metric, F.Cu at (121.0, 82.6)
- added C32: 10uF, PCM_SparkFun-Capacitor:C_0805_2012Metric, F.Cu at (124.7, 82.3)
- added C33: 100uF, PCM_SparkFun-Capacitor:Panasonic_D, F.Cu at (130.5, 80.7)
- added C34: 470uF, PCM_SparkFun-Capacitor:Electrolytic_10.3x10.3mm, F.Cu at (140.2, 80.6)
- added C35: 0.1uF, PCM_SparkFun-Capacitor:C_0603_1608Metric, F.Cu at (128.2, 31.1)
- added C36: 100uF, PCM_SparkFun-Capacitor:Panasonic_D, F.Cu at (118.2, 107.1)
- added C37: 0.1uF, PCM_SparkFun-Capacitor:C_0603_1608Metric, F.Cu at (123.2, 34.6)
- added C39: 0.1uF, PCM_SparkFun-Capacitor:C_0603_1608Metric, F.Cu at (125.7, 32.1)
- added C40: 1.0uF, PCM_SparkFun-Capacitor:C_0402_1005Metric, F.Cu at (116.2, 101.1)
- added C42: 10uF, PCM_SparkFun-Capacitor:C_0805_2012Metric, F.Cu at (120.0, 101.1)
- added C43: 100uF, PCM_SparkFun-Capacitor:Panasonic_D, F.Cu at (126.5, 100.6)
- added C44: 470uF, PCM_SparkFun-Capacitor:Electrolytic_10.3x10.3mm, F.Cu at (136.8, 100.6)
- added C45: 470uF, PCM_SparkFun-Capacitor:Electrolytic_10.3x10.3mm, F.Cu at (137.2, 163.5)
- added C46: 100uF, PCM_SparkFun-Capacitor:C_1206_3216Metric, F.Cu at (124.8, 145.8)
- added C47: 100uF, PCM_SparkFun-Capacitor:C_1206_3216Metric, F.Cu at (111.1, 145.8)
- added C48: 100uF, PCM_SparkFun-Capacitor:C_1206_3216Metric, F.Cu at (137.6, 144.0)
- added D10: 1N5822, Diode_THT:D_DO-201AD_P15.24mm_Horizontal, F.Cu at (153.1, 149.8)
- added D8: 1N5822, Diode_THT:D_DO-201AD_P15.24mm_Horizontal, F.Cu at (88.7, 148.2)
- added D9: 1N5822, Diode_THT:D_DO-201AD_P15.24mm_Horizontal, F.Cu at (113.8, 151.0)
- added J13: 3.5mm, PCM_SparkFun-Connector:ScrewTerminal_1x02_P3.5mm_Horizontal_Black, F.Cu at (100.6, 159.2)
- added L5: 4.7uH, PCM_SparkFun-Coil:1008_2520Metric, F.Cu at (118.2, 145.8)
- added L6: 4.7uH, PCM_SparkFun-Coil:1008_2520Metric, F.Cu at (134.8, 154.8)
- added LS1: Speaker, Connector:JWT_A3963_1x02_P3.96mm_Vertical, F.Cu at (99.4, 85.0)
- added LS3: Speaker, Connector:JWT_A3963_1x02_P3.96mm_Vertical, F.Cu at (89.1, 85.0)
- added M3: Stepper_Motor_bipolar, Connector_PinHeader_2.54mm:PinHeader_1x04_P2.54mm_Vertical, F.Cu at (112.2, 91.1)
- added M4: Stepper_Motor_bipolar, Connector_PinHeader_2.54mm:PinHeader_1x04_P2.54mm_Vertical, F.Cu at (124.5, 108.0)
- added MK1: INMP441ACEZ-R7, SnapEDA_Footprints:MIC_INMP441ACEZ-R7, F.Cu at (102.0, 110.3)
- added MK2: INMP441ACEZ-R7, SnapEDA_Footprints:MIC_INMP441ACEZ-R7, F.Cu at (92.1, 110.3)
- added U10-TMC-R1: TMC2209-LA, Package_DFN_QFN:VQFN-28-1EP_5x5mm_P0.5mm_EP3.7x3.7mm_ThermalVias, F.Cu at (131.8, 112.3)
- added U11-IMU1: ICM-20948, Sensor_Motion:InvenSense_QFN-24_3x3mm_P0.4mm, F.Cu at (124.7, 28.4)
- added U12-LM-adj1: LM2596S-ADJ, Package_TO_SOT_SMD:TO-263-5_TabPin3, F.Cu at (104.5, 131.9)
- added U13-LM-12: LM2596S-12, Package_TO_SOT_SMD:TO-263-5_TabPin3, F.Cu at (119.3, 132.1)
- added U14-LM-5: LM2596S-5, Package_TO_SOT_SMD:TO-263-5_TabPin3, F.Cu at (134.3, 131.8)
- added U9-TMC-L1: TMC2209-LA, Package_DFN_QFN:VQFN-28-1EP_5x5mm_P0.5mm_EP3.7x3.7mm_ThermalVias, F.Cu at (119.8, 88.6)
- C1, C4: value 100uF -> 10uF; footprint PCM_SparkFun-Capacitor:Panasonic_D -> PCM_SparkFun-Capacitor:C_0402_1005Metric
- C2: value 100uF -> 0.1uF; footprint PCM_SparkFun-Capacitor:Panasonic_D -> Capacitor_SMD:C_01005_0402Metric
- C3: value 10uF -> 0.1uF; footprint PCM_SparkFun-Capacitor:C_0603_1608Metric_Polar -> PCM_SparkFun-Capacitor:C_0402_1005Metric
- C5: value 2.2uF -> 0.1uF; footprint PCM_SparkFun-Capacitor:C_0805_2012Metric -> PCM_SparkFun-Capacitor:C_0402_1005Metric
- C6: value 100uF -> 0.1uF; footprint PCM_SparkFun-Capacitor:Panasonic_D -> PCM_SparkFun-Capacitor:C_0402_1005Metric
- C7: value 1uF_0603_25V -> 470nF; footprint PCM_4ms_Capacitor:C_0603 -> PCM_SparkFun-Capacitor:C_0201_0603Metric
- C8: value 47uF -> 470nF; footprint PCM_SparkFun-Capacitor:C_0805_2012Metric -> PCM_SparkFun-Capacitor:C_0201_0603Metric
- D1: footprint PCM_Diode_THT_AKL:D_DO-201AD_P12.70mm_Horizontal -> Diode_THT:D_DO-201AD_P15.24mm_Horizontal
- F2: value Fuse_Polarized -> Fuse; footprint Fuse:Fuse_0402_1005Metric -> Fuse:Fuse_0603_1608Metric
- J1: footprint Connector_Harwin:Harwin_M20-89005xx_1x05_P2.54mm_Horizontal -> Connector_Hirose:Hirose_DF13-05P-1.25DSA_1x05_P1.25mm_Vertical
- J2: value Conn_01x06_Pin -> Barrel_Jack_MountingPin; footprint Connector_Harwin:Harwin_M20-89006xx_1x06_P2.54mm_Horizontal -> Connector_BarrelJack:BarrelJack_CUI_PJ-063AH_Horizontal_CircularHoles
- J9: value Conn_01x01_Pin -> Conn_01x02_Pin; footprint Connector_PinHeader_1.00mm:PinHeader_1x01_P1.00mm_Vertical -> Connector:JWT_A3963_1x02_P3.96mm_Vertical
- L4: value 1.0uH -> 4.7uH; footprint PCM_SparkFun-Coil:0805 -> PCM_SparkFun-Coil:1008_2520Metric
- R1: value 3.3k -> 10k
- R10: value 4.7k -> 100k; footprint PCM_SparkFun-Resistor:R_0402_1005Metric -> PCM_SparkFun-Resistor:R_0603_1608Metric
- R2: value 3.3k -> 4.7k
- R7: value 10k_0402 -> 100k; footprint Resistor_SMD:R_0402_1005Metric -> PCM_SparkFun-Resistor:R_0603_1608Metric
- R8: value 10k_0402 -> 10k; footprint Resistor_SMD:R_0402_1005Metric -> PCM_SparkFun-Resistor:R_0603_1608Metric
- R9: value 4.7k -> 10k; footprint PCM_SparkFun-Resistor:R_0402_1005Metric -> PCM_SparkFun-Resistor:R_0603_1608Metric
- U1: value LM2596S-ADJ -> MAX98357A; footprint Package_TO_SOT_SMD:TO-263-5_TabPin3 -> Package_DFN_QFN:TQFN-16-1EP_3x3mm_P0.5mm_EP1.23x1.23mm_ThermalVias
- U2: value LM2596S-5 -> MAX98357A; footprint PCM_Package_TO_SOT_SMD_AKL:TO-263-4_ThermalVias -> Package_DFN_QFN:TQFN-16-1EP_3x3mm_P0.5mm_EP1.23x1.23mm
- moved D1 135.2 mm to (112.6, 160.0)
- moved F2 116.9 mm to (108.3, 157.5)
- moved C1 91.2 mm to (92.5, 99.2)
- moved C6 85.8 mm to (91.2, 115.5), turned to 180 degrees
- moved C2 85.1 mm to (88.0, 95.4), turned to -90 degrees
- moved R2 80.4 mm to (99.5, 107.5), turned to 180 degrees
- moved J1 77.5 mm to (94.2, 103.2)
- moved R1 77.4 mm to (96.8, 96.2)
- moved J9 73.8 mm to (94.6, 70.6)
- moved C4 69.5 mm to (104.0, 96.7), turned to 90 degrees
- moved C3 66.7 mm to (100.8, 99.5)
- moved J2 64.1 mm to (91.6, 158.8)
- moved R10 61.7 mm to (138.0, 111.7), turned to 90 degrees
- moved L4 60.5 mm to (108.0, 148.2)
- moved R7 55.2 mm to (125.8, 86.8), turned to 90 degrees
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Connections:
- A2 pad 12: Net-(A2-GPIO9) -> unconnected-(A2-GPIO9-Pad12)_1
- A2 pad 13: GNDPWR -> GND
- A2 pad 18: GNDPWR -> GND
- A2 pad 23: GNDPWR -> GND
- A2 pad 25: unconnected-(A2-GPIO19-Pad25) -> Net-(A2-GPIO19)
- A2 pad 28: GNDPWR -> GND
- A2 pad 3: GNDPWR -> GND
- A2 pad 36: Net-(A2-3V3) -> 3.3V
- A2 pad 38: GNDPWR -> GND
- A2 pad 39: Net-(A2-VSYS) -> 5V
- A2 pad 7: Net-(A2-GPIO5) -> unconnected-(A2-GPIO5-Pad7)
- A2 pad 8: GNDPWR -> GND
- C1 pad 1: Net-(J1-Pin_1) -> 5V
- C2 pad 1: Net-(J1-Pin_1) -> 5V
- C3 pad 1: Net-(A1-VSYS) -> 5V
- C4 pad 1: Net-(D1-A) -> 5V
- C5 pad 1: Net-(D1-A) -> 3.3V
- C6 pad 1: Net-(J10-Pin_1) -> 3.3V
- C7 pad 1: Net-(J10-Pin_1) -> 12V
- C7 pad 2: GND -> Net-(U9-TMC-L1-VCP)
- C8 pad 1: Net-(J10-Pin_1) -> 12V
- C8 pad 2: GND -> Net-(U10-TMC-R1-VCP)
- F2 pad 2: GND -> Net-(D1-A)
- J1 pad 2: GND -> Net-(J1-Pin_2)
- J1 pad 3: Net-(A1-GPIO1) -> Net-(J1-Pin_3)
- J1 pad 4: Net-(A1-GPIO0) -> Net-(J1-Pin_4)
- J1 pad 5: Net-(A1-VSYS) -> Net-(J1-Pin_5)
- J2 pad 1: Net-(J2-Pin_1) -> Net-(U12-LM-adj1-FB)
- J2 pad 2: Net-(J2-Pin_2) -> GND
- J9 pad 1: Net-(J9-Pin_1) -> Net-(A2-GPIO0)
- L4 pad 2: Net-(J8-Pin_1) -> Net-(U12-LM-adj1-FB)
- R1 pad 1: Net-(U7-~{SD_MODE}) -> GND
- R1 pad 2: Net-(J2-Pin_5) -> Net-(J1-Pin_3)
- R10 pad 1: Net-(A2-GPIO16) -> GND
- R2 pad 2: Net-(J4-Pin_5) -> Net-(J1-Pin_4)
- R7 pad 1: Net-(A2-GPIO4) -> GND
- R8 pad 1: Net-(A2-GPIO8) -> Net-(A2-GPIO16)
- U1 pad 1: Net-(D1-A) -> Net-(J1-Pin_5)
- U1 pad 2: Net-(D2-A) -> 5V
- U1 pad 4: Net-(J10-Pin_1) -> Net-(J1-Pin_3)
- U1 pad 5: GND -> unconnected-(U1-NC-Pad5)
- U2 pad 1: Net-(D1-A) -> Net-(J1-Pin_5)
- U2 pad 2: Net-(D3-A) -> 5V
- U2 pad 4: Net-(J9-Pin_1) -> Net-(J1-Pin_3)
- U2 pad 5: GND -> unconnected-(U2-NC-Pad5)
Routing:
- net 12V: track 0.00 -> 318.0 mm
- net Net-(J1-Pin_2): track 0.00 -> 179.9 mm
- net 3.3V: track 0.00 -> 113.9 mm
- net 5V: track 0.00 -> 110.2 mm
- net Net-(D1-A): track 0.00 -> 83.8 mm
- net Net-(J1-Pin_1): track 0.00 -> 72.8 mm
- net Net-(A2-GPIO2): track 0.00 -> 71.5 mm
- net Net-(U10-TMC-R1-VCP): track 0.00 -> 53.2 mm
- net Net-(A2-GPIO3): track 0.00 -> 37.9 mm
- net Net-(U1-OUTP): track 0.00 -> 34.8 mm
- net Net-(D10-A): track 0.00 -> 33.7 mm
- net Net-(U12-LM-adj1-FB): track 0.00 -> 33.6 mm
- net Net-(J1-Pin_3): track 0.00 -> 29.7 mm
- net Net-(A2-GPIO16): track 0.00 -> 28.8 mm
- net Net-(A2-GPIO18): track 0.00 -> 28.4 mm
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- added copper zone on In1.Cu, net GND
Other:
- board outline added: 75.8 x 153 mm
- copper layers 2 -> 4
- board text added: "IMU Sensor"
- board text added: "Left"
- board text added: "Mic-Speaker"
- board text added: "Power Supply"
- board text added: "Right"
- board text added: "Stepper Motors"
