File: Schematics-PCB-Design/aadhuNIK-Main/_restore_backup_2026-05-28T11-59-53-382/aadhuNIK-Main.kicad_sch (KiCad schematic)
At the start: 58 parts, among them J1 Conn_01x05_Pin, J13 3.5mm, J2 Barrel_Jack_MountingPin, J9 Conn_01x02_Pin, M3 Stepper_Motor_bipolar, M4 Stepper_Motor_bipolar, U1 MAX98357A, U10-TMC-R1 TMC2209-LA, U11-IMU1 ICM-20948, U12-LM-adj1 LM2596S-ADJ, U13-LM-12 LM2596S-12, U14-LM-5 LM2596S-5, U2 MAX98357A, U9-TMC-L1 TMC2209-LA

Commit message: Update KiCad schematic and PCB
Parts:
- removed C7, C8: 470nF, PCM_SparkFun-Capacitor:C_0201_0603Metric, symbol PCM_SparkFun-Capacitor:470nF_0201_6.3V_20%
- removed D1: 1N5822, Diode_THT:D_DO-201AD_P15.24mm_Horizontal, symbol Diode:1N5822
- removed J2: Barrel_Jack_MountingPin, Connector_BarrelJack:BarrelJack_CUI_PJ-063AH_Horizontal_CircularHoles, symbol Connector:Barrel_Jack_MountingPin
- removed LS3: Speaker, Connector:JWT_A3963_1x02_P3.96mm_Vertical, symbol Device:Speaker
- removed U10-TMC-R1, U9-TMC-L1: TMC2209-LA, Package_DFN_QFN:VQFN-28-1EP_5x5mm_P0.5mm_EP3.7x3.7mm_ThermalVias, symbol Driver_Motor:TMC2209-LA
- removed U11-IMU1: ICM-20948, Sensor_Motion:InvenSense_QFN-24_3x3mm_P0.4mm, symbol Sensor_Motion:ICM-20948
- removed U12-LM-adj1: LM2596S-ADJ, Package_TO_SOT_SMD:TO-263-5_TabPin3, symbol Regulator_Switching:LM2596S-ADJ
- removed U13-LM-12: LM2596S-12, Package_TO_SOT_SMD:TO-263-5_TabPin3, symbol Regulator_Switching:LM2596S-12
- removed U14-LM-5: LM2596S-5, Package_TO_SOT_SMD:TO-263-5_TabPin3, symbol Regulator_Switching:LM2596S-5
- added C29, C31, C38, C41: 100uF, PCM_SparkFun-Capacitor:Panasonic_D, symbol PCM_SparkFun-Capacitor:100uF_6.6x6.6_25V_20%
- added D6, D7: 1N5822, Diode_THT:D_DO-201AD_P15.24mm_Horizontal, symbol Diode:1N5822
- added J10: Conn_01x01_Pin, Connector_Hirose:Hirose_DF63M-1P-3.96DSA_1x01_P3.96mm_Vertical, symbol Connector:Conn_01x01_Pin
- added J14: 3.5mm, PCM_SparkFun-Connector:ScrewTerminal_1x04_P3.5mm_Horizontal, symbol PCM_SparkFun-Connector:ScrewTerminal_1x04_P3.5mm_Horizontal
- added J2: 3.5mm, PCM_SparkFun-Connector:ScrewTerminal_1x03_P3.5mm_Horizontal_Black, symbol PCM_SparkFun-Connector:ScrewTerminal_1x03_P3.5mm_Horizontal_Black
- added LS2: Speaker, Battery:BatteryHolder_Bulgin_BX0034_1xAAA, symbol Device:Speaker
- added U10, U9: TMC2209-LA, Package_DFN_QFN:VQFN-28-1EP_5x5mm_P0.5mm_EP3.7x3.7mm_ThermalVias, symbol Driver_Motor:TMC2209-LA
- added U11: ICM-20948, Sensor_Motion:InvenSense_QFN-24_3x3mm_P0.4mm, symbol Sensor_Motion:ICM-20948
- added U12: LM2596S-ADJ, Package_TO_SOT_SMD:TO-263-5_TabPin3, symbol Regulator_Switching:LM2596S-ADJ
- added U13: LM2596S-12, Package_TO_SOT_SMD:TO-263-5_TabPin3, symbol Regulator_Switching:LM2596S-12
- added U14: LM2596S-5, Package_TO_SOT_SMD:TO-263-5_TabPin3, symbol Regulator_Switching:LM2596S-5
- LS1: footprint Connector:JWT_A3963_1x02_P3.96mm_Vertical -> Battery:BatteryHolder_Bulgin_BX0034_1xAAA
Connections:
- net 3.3V: now also J2.3 (Pin_3); no longer A2.36 (3V3), C28.1, C35.1, C36.1, C37.1
- net 5V: now also J14.3 (Pin_3), J2.1 (Pin_1), U14.4 (FB); no longer A2.39 (VSYS)
- net GND: now also A2.33 (AGND), R2.1, D7.1 (K), J14.4 (Pin_4), J2.2 (Pin_2), U10.18 (GND), U10.29 (GND), U10.3 (GND), U11.18 (GND), U11.20 (GND), U12.3 (GND), U12.5 (~{ON}/OFF), U13.3 (GND), U13.5 (~{ON}/OFF), U14.3 (GND), U14.5 (~{ON}/OFF), U9.18 (GND), U9.29 (GND), U9.3 (GND); no longer A2.13 (GND), A2.18 (GND), A2.23 (GND), A2.28 (GND), A2.3 (GND), A2.38 (GND), A2.8 (GND)
- net at C47.1, L4.2: now also J14.1 (Pin_1), U12.4 (FB)
- net at D8.2 (A), L4.1: now also U12.2 (OUT)
- net at M4.1: now also U10.24 (OA1)
- net at M4.2 (-): now also U10.21 (OA2)
- net at M4.3: now also U10.26 (OB1)
- net at M4.4: now also U10.1 (OB2)
- net at C45.1, F2.2: now also D7.2 (A), U12.1 (VIN), U13.1 (VIN), U14.1 (VIN)
- net at U1.10 (OUTN): now also LS2.2
- net at U1.9 (OUTP): now also LS2.1
- net at C39.1: now also U11.10 (REGOUT)
- net at D10.2 (A), L6.1: now also U14.2 (OUT)
- net at D9.2 (A), L5.1: now also U13.2 (OUT)
- net at R8.2: now also U11.24 (SDA/SDI)
- net at A2.9 (GPIO6): now also U10.16 (STEP)
- net at A2.10 (GPIO7): now also U10.19 (DIR)
- net at A2.11 (GPIO8): now also U10.2 (~{EN})
- net at R10.2: now also U10.20 (STDBY)
- net at M3.4: now also U9.1 (OB2)
- net at A2.4 (GPIO2): now also U9.16 (STEP)
- net at A2.5 (GPIO3): now also U9.19 (DIR)
- net at A2.6 (GPIO4): now also U9.2 (~{EN})
- net at R7.2: now also U9.20 (STDBY)
- net at M3.2 (-): now also U9.21 (OA2)
- net at M3.1: now also U9.24 (OA1)
- net at M3.3: now also U9.26 (OB1)
- net at MK1.2 (SD): now also J1.4 (Pin_4), MK2.2 (SD), R2.2; no longer R2.1
- net at A2.12 (GPIO9): now also U10.14 (~{PD}/UART)
- net at A2.24 (GPIO18): now also U11.9 (SDO/AD0)
- net at A2.25 (GPIO19): now also U11.12 (INT1)
- net at A2.7 (GPIO5): now also U9.14 (~{PD}/UART)
- net at R9.2: now also U11.23 (SCL/SCLK)
- net 12V: no longer names the net of C30.1, C32.1, C33.1, C34.1, C40.1, C42.1, C43.1, C44.1, C46.1, L5.2
- net 12V: now also C29.1, C38.1, J14.2 (Pin_2), U10.22 (VS), U10.28 (VS), U13.4 (FB), U9.22 (VS), U9.28 (VS)
- new net: A2.36 (3V3), C28.1, C35.1, C36.1, C37.1, U10.15 (VCC_IO), U11.13 (VDD), U11.22 (~{CS}), U11.8 (VDDIO), U9.15 (VCC_IO)
- new net: C38.2, U10.6 (VCP)
- new net: D6.1 (K), J10.1 (Pin_1)
- new net: A2.39 (VSYS), D6.2 (A)
- new net: C31.1, U9.4 (CPO)
- new net: C31.2, U9.5 (CPI)
- new net: C29.2, U9.6 (VCP)
- new net: A2.13 (GND), A2.18 (GND), A2.23 (GND), A2.28 (GND), A2.3 (GND), A2.38 (GND), A2.8 (GND)
- new net: C41.1, U10.4 (CPO)
- new net: C41.2, U10.5 (CPI)
- no-connect marks 53 -> 44
