File: Schematics-PCB-Design/aadhuNIK-Main/_restore_backup_2026-05-28T14-14-27-077/aadhuNIK-Main.kicad_sch (KiCad schematic)
At the start: 58 parts, among them J1 Conn_01x05_Pin, J13 3.5mm, J2 Barrel_Jack_MountingPin, J9 Conn_01x02_Pin, M3 Stepper_Motor_bipolar, M4 Stepper_Motor_bipolar, U1 MAX98357A, U10-TMC-R1 TMC2209-LA, U11-IMU1 ICM-20948, U12-LM-adj1 LM2596S-ADJ, U13-LM-12 LM2596S-12, U14-LM-5 LM2596S-5, U2 MAX98357A, U9-TMC-L1 TMC2209-LA

Commit message: Update KiCad schematic and PCB
Parts:
- removed D1: 1N5822, Diode_THT:D_DO-201AD_P15.24mm_Horizontal, symbol Diode:1N5822
- removed J2: Barrel_Jack_MountingPin, Connector_BarrelJack:BarrelJack_CUI_PJ-063AH_Horizontal_CircularHoles, symbol Connector:Barrel_Jack_MountingPin
- added C31, C41: 100uF, PCM_SparkFun-Capacitor:Panasonic_D, symbol PCM_SparkFun-Capacitor:100uF_6.6x6.6_25V_20%
- added D6, D7: 1N5822, Diode_THT:D_DO-201AD_P15.24mm_Horizontal, symbol Diode:1N5822
- added J10: Conn_01x01_Pin, Connector_Hirose:Hirose_DF63M-1P-3.96DSA_1x01_P3.96mm_Vertical, symbol Connector:Conn_01x01_Pin
- added J14: 3.5mm, PCM_SparkFun-Connector:ScrewTerminal_1x04_P3.5mm_Horizontal, symbol PCM_SparkFun-Connector:ScrewTerminal_1x04_P3.5mm_Horizontal
- added J2: 3.5mm, PCM_SparkFun-Connector:ScrewTerminal_1x03_P3.5mm_Horizontal_Black, symbol PCM_SparkFun-Connector:ScrewTerminal_1x03_P3.5mm_Horizontal_Black
Connections:
- net 3.3V: now also J2.3 (Pin_3); no longer A2.36 (3V3), C28.1, C35.1, C36.1, C37.1, U10-TMC-R1.15 (VCC_IO), U11-IMU1.13 (VDD), U11-IMU1.22 (~{CS}), U11-IMU1.8 (VDDIO), U9-TMC-L1.15 (VCC_IO)
- net 5V: now also J14.3 (Pin_3), J2.1 (Pin_1); no longer A2.39 (VSYS)
- net GND: now also R2.1, D7.1 (K), J14.4 (Pin_4), J2.2 (Pin_2)
- net at C47.1, L4.2, U12-LM-adj1.4 (FB): now also J14.1 (Pin_1)
- net at C45.1, F2.2, U12-LM-adj1.1 (VIN)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: now also D7.2 (A)
- net at U10-TMC-R1.14 (~{PD}/UART): now also A2.12 (GPIO9)
- net at U10-TMC-R1.4 (CPO): now also C41.1
- net at U10-TMC-R1.5 (CPI): now also C41.2
- net at U9-TMC-L1.14 (~{PD}/UART): now also A2.7 (GPIO5)
- net at U9-TMC-L1.4 (CPO): now also C31.1
- net at U9-TMC-L1.5 (CPI): now also C31.2
- net at MK1.2 (SD): now also J1.4 (Pin_4), MK2.2 (SD), R2.2; no longer R2.1
- net 12V: no longer names the net of C30.1, C32.1, C33.1, C34.1, C40.1, C42.1, C43.1, C44.1, C46.1, C7.1, C8.1, L5.2, U10-TMC-R1.22 (VS), U10-TMC-R1.28 (VS), U13-LM-12.4 (FB), U9-TMC-L1.22 (VS), U9-TMC-L1.28 (VS)
- net 12V: now also J14.2 (Pin_2)
- new net: A2.36 (3V3), C28.1, C35.1, C36.1, C37.1, U10-TMC-R1.15 (VCC_IO), U11-IMU1.13 (VDD), U11-IMU1.22 (~{CS}), U11-IMU1.8 (VDDIO), U9-TMC-L1.15 (VCC_IO)
- new net: D6.1 (K), J10.1 (Pin_1)
- new net: A2.39 (VSYS), D6.2 (A)
- no-connect marks 53 -> 44
