File: Schematics-PCB-Design/aadhuNIKai/aadhuNIKai.kicad_sch (KiCad schematic)
At the start: 58 parts, among them J1 Conn_01x05_Pin, J13 3.5mm, J2 Barrel_Jack_MountingPin, J9 Conn_01x02_Pin, M3 Stepper_Motor_bipolar, M4 Stepper_Motor_bipolar, U1 MAX98357A, U10-TMC-R1 TMC2209-LA, U11-IMU1 ICM-20948, U12-LM-adj1 LM2596S-ADJ, U13-LM-12 LM2596S-12, U14-LM-5 LM2596S-5, U2 MAX98357A, U9-TMC-L1 TMC2209-LA

Commit message: Update KiCad schematic and PCB
Parts:
- removed D1: 1N5822, Diode_THT:D_DO-201AD_P15.24mm_Horizontal, symbol Diode:1N5822
- added C31, C41: 100uF, PCM_SparkFun-Capacitor:Panasonic_D, symbol PCM_SparkFun-Capacitor:100uF_6.6x6.6_25V_20%
- added D7: 1N5822, Diode_THT:D_DO-201AD_P15.24mm_Horizontal, symbol Diode:1N5822
Connections:
- net GND: now also D7.1 (K)
- net VIN: now reaches C45.1, F2.2, U12-LM-adj1.1 (VIN), U13-LM-12.1 (VIN), U14-LM-5.1 (VIN)
- net VIN: now also D7.2 (A)
- net at U10-TMC-R1.4 (CPO): now also C41.1
- net at U10-TMC-R1.5 (CPI): now also C41.2
- net at U9-TMC-L1.4 (CPO): now also C31.1
- net at U9-TMC-L1.5 (CPI): now also C31.2
- net 12V: no longer names the net of C30.1, C32.1, C33.1, C34.1, C40.1, C42.1, C43.1, C44.1, C46.1, C7.1, C8.1, L5.2, U10-TMC-R1.22 (VS), U10-TMC-R1.28 (VS), U13-LM-12.4 (FB), U9-TMC-L1.22 (VS), U9-TMC-L1.28 (VS)
- no-connect marks 53 -> 48
Other:
- company: Aadhunik AI  -> (none)
